File: CAD/integrator-V6.kicad_sch (KiCad schematic)
At the start: 36 parts, among them J1 Screw_Terminal_01x03, J2 Barrel_Jack_Switch, J3 AudioJack2_Ground_Switch, SW1 SW_SPDT_MSM, U1 TL084, U2 L78L06_SOT89

Commit message: Add files via upload
Parts:
- renumbered R4 to R3, R3 to R4
Changed lines of the file:
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@@
 		(on_board yes)
 		(dnp no)
-		(property "Reference" "R3"
+		(property "Reference" "R4"
 			(at 108.585 110.49 0)
 			(effects
@@
 			(project "integrator-V6"
 				(path "/b7263ebf-d74d-4fdb-8017-e4e8544e3c77"
-					(reference "R3")
+					(reference "R4")
 					(unit 1)
 				)
@@
 		(dnp no)
 		(fields_autoplaced yes)
-		(property "Reference" "R4"
+		(property "Reference" "R3"
 			(at 109.22 69.215 0)
 			(effects
@@
 			(project "integrator-V6"
 				(path "/b7263ebf-d74d-4fdb-8017-e4e8544e3c77"
-					(reference "R4")
-					(unit 1)
-				)
+					(reference "R3")
+					(unit 1)
+				)
